File: misguided/npu.kicad_sch (KiCad schematic)
At the start: 0 parts

Commit message: buncha stuff
Other:
- note added: "Use the M.2 M key"
- note removed: "Use the M.2 Connector version"
Changed lines of the file:
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@@
 (kicad_sch (version 20230121) (generator eeschema)
   (paper "A4")
-  (text "Use the M.2 Connector version\n\n" (at 72.898 55.372 0)
+  (text "Use the M.2 M key\n\n" (at 72.898 55.372 0)
     (effects (font (size 1.27 1.27)) (justify left bottom))
   )
+  (hierarchical_label "PCIE_TX_P" (shape output) (at 80.645 72.39 180) (fields_autoplaced)
+    (effects (font (size 1.27 1.27)) (justify right))
+  )
+  (hierarchical_label "PCIE_RX_P" (shape input) (at 80.645 66.675 180) (fields_autoplaced)
+    (effects (font (size 1.27 1.27)) (justify right))
+  )
+  (hierarchical_label "PCIE_CLKREQ_N" (shape input) (at 80.645 83.82 180) (fields_autoplaced)
+    (effects (font (size 1.27 1.27)) (justify right))
+  )
+  (hierarchical_label "PCIE_RST_B" (shape input) (at 80.01 86.36 180) (fields_autoplaced)
+    (effects (font (size 1.27 1.27)) (justify right))
+  )
+  (hierarchical_label "PCIE_DET_WAKE" (shape input) (at 80.645 81.28 180) (fields_autoplaced)
+    (effects (font (size 1.27 1.27)) (justify right))
+  )
+  (hierarchical_label "PCIE_PWR_EN" (shape input) (at 80.645 79.375 180) (fields_autoplaced)
+    (effects (font (size 1.27 1.27)) (justify right))
+  )
+  (hierarchical_label "PCIE_CLK_N" (shape input) (at 80.645 62.23 180) (fields_autoplaced)
+    (effects (font (size 1.27 1.27)) (justify right))
+  )
+  (hierarchical_label "PCIE_CLK_P" (shape input) (at 80.645 60.325 180) (fields_autoplaced)
+    (effects (font (size 1.27 1.27)) (justify right))
+  )
+  (hierarchical_label "PCIE_RX_N" (shape input) (at 80.645 68.58 180) (fields_autoplaced)
+    (effects (font (size 1.27 1.27)) (justify right))
+  )
+  (hierarchical_label "PCIE_TX_N" (shape output) (at 80.645 74.295 180) (fields_autoplaced)
+    (effects (font (size 1.27 1.27)) (justify right))
+  )
 )
