File: misguided/misguided.kicad_sch (KiCad schematic)
At the start: 3 parts, among them J101 Conn_01x03, J102 Conn_01x03, J103 Conn_01x03

Commit message: buncha stuff
Parts:
- added J104: Conn_01x16, Connector_FFC-FPC:TE_1-1734839-6_1x16-1MP_P0.5mm_Horizontal, symbol Connector_Generic:Conn_01x16
Changed lines of the file:
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@@
+    )
+  )
+  (symbol (lib_id "Connector_Generic:Conn_01x16") (at 44.45 151.765 0) (mirror y) (unit 1)
+    (in_bom yes) (on_board yes) (dnp no) (fields_autoplaced)
+    (property "Reference" "J104" (at 44.45 128.27 0)
+      (effects (font (size 1.27 1.27)))
+    )
+    (property "Value" "Conn_01x16" (at 44.45 130.81 0)
+      (effects (font (size 1.27 1.27)))
+    )
+    (property "Footprint" "Connector_FFC-FPC:TE_1-1734839-6_1x16-1MP_P0.5mm_Horizontal" (at 44.45 151.765 0)
+      (effects (font (size 1.27 1.27)) hide)
+    )
+    (property "Datasheet" "~" (at 44.45 151.765 0)
+      (effects (font (size 1.27 1.27)) hide)
+    )
+    (pin "1")
+    (pin "10")
+    (pin "11")
+    (pin "12")
+    (pin "13")
+    (pin "14")
+    (pin "15")
+    (pin "16")
+    (pin "2")
+    (pin "3")
+    (pin "4")
+    (pin "5")
+    (pin "6")
+    (pin "7")
+    (pin "8")
+    (pin "9")
+    (instances
+      (project "misguided"
+        (path "/2c6152e0-1c3c-4f15-8d1e-fd42bd51bc79"
+          (reference "J104") (unit 1)
+        )
+      )
     )
   )

Commit message: more setup
Parts:
- removed J104: Conn_01x16, Connector_FFC-FPC:TE_1-1734839-6_1x16-1MP_P0.5mm_Horizontal, symbol Connector_Generic:Conn_01x16
- added M101: ~, misguided:pi_hat, symbol misguided:hat+
Other:
- removed sheet npu
Changed lines of the file:
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@@
-    )
-  )
-  (symbol (lib_id "Connector_Generic:Conn_01x16") (at 44.45 151.765 0) (mirror y) (unit 1)
-    (in_bom yes) (on_board yes) (dnp no) (fields_autoplaced)
-    (property "Reference" "J104" (at 44.45 128.27 0)
-      (effects (font (size 1.27 1.27)))
-    )
-    (property "Value" "Conn_01x16" (at 44.45 130.81 0)
-      (effects (font (size 1.27 1.27)))
-    )
-    (property "Footprint" "Connector_FFC-FPC:TE_1-1734839-6_1x16-1MP_P0.5mm_Horizontal" (at 44.45 151.765 0)
-      (effects (font (size 1.27 1.27)) hide)
-    )
-    (property "Datasheet" "~" (at 44.45 151.765 0)
-      (effects (font (size 1.27 1.27)) hide)
-    )
-    (pin "1")
-    (pin "10")
-    (pin "11")
-    (pin "12")
-    (pin "13")
-    (pin "14")
-    (pin "15")
-    (pin "16")
-    (pin "2")
-    (pin "3")
-    (pin "4")
-    (pin "5")
-    (pin "6")
-    (pin "7")
-    (pin "8")
-    (pin "9")
-    (instances
-      (project "misguided"
-        (path "/2c6152e0-1c3c-4f15-8d1e-fd42bd51bc79"
-          (reference "J104") (unit 1)
-        )
-      )
     )
   )
@@
         (path "/2c6152e0-1c3c-4f15-8d1e-fd42bd51bc79"
           (reference "J102") (unit 1)
+        )
+      )
+    )
+  )
+  (symbol (lib_id "misguided:hat+") (at 50.165 42.545 0) (unit 1)
+    (in_bom yes) (on_board yes) (dnp no) (fields_autoplaced)
+    (property "Reference" "M101" (at 50.165 41.91 0)
+      (effects (font (size 1.27 1.27)))
+    )
+    (property "Value" "~" (at 53.34 42.545 0)
+      (effects (font (size 1.27 1.27)) hide)
+    )
+    (property "Footprint" "misguided:pi_hat" (at 53.34 42.545 0)
+      (effects (font (size 1.27 1.27)) hide)
+    )
+    (property "Datasheet" "${KIPRJMOD}/datasheets/hat-plus-specification.pdf" (at 53.34 42.545 0)
+      (effects (font (size 1.27 1.27)) hide)
+    )
+    (pin "1")
+    (pin "10")
+    (pin "11")
+    (pin "12")
+    (pin "13")
+    (pin "14")
+    (pin "15")
+    (pin "16")
+    (pin "17")
+    (pin "18")
+    (pin "19")
+    (pin "2")
+    (pin "20")
+    (pin "21")
+    (pin "22")
+    (pin "23")
+    (pin "24")
+    (pin "25")
+    (pin "26")
+    (pin "27")
+    (pin "28")
+    (pin "29")
+    (pin "3")
+    (pin "30")
+    (pin "31")
+    (pin "32")
+    (pin "33")
+    (pin "34")
+    (pin "35")
+    (pin "36")
+    (pin "37")
+    (pin "38")
+    (pin "39")
+    (pin "4")
+    (pin "40")
+    (pin "5")
+    (pin "6")
+    (pin "7")
+    (pin "8")
+    (pin "9")
+    (pin "SH")
+    (instances
+      (project "misguided"
+        (path "/2c6152e0-1c3c-4f15-8d1e-fd42bd51bc79"
+          (reference "M101") (unit 1)
         )
       )
@@
       )
     )
-  )
-  (sheet (at 110.744 140.462) (size 48.006 17.78) (fields_autoplaced)
-    (stroke (width 0.1524) (type solid))
-    (fill (color 0 0 0 0.0000))
-    (property "Sheetname" "npu" (at 110.744 139.7504 0)
-      (effects (font (size 1.27 1.27)) (justify left bottom))
-    )
-    (property "Sheetfile" "npu.kicad_sch" (at 110.744 158.8266 0)
-      (effects (font (size 1.27 1.27)) (justify left top))
-    )
-    (instances
-      (project "misguided"
-        (path "/2c6152e0-1c3c-4f15-8d1e-fd42bd51bc79" (page "5"))
-      )
-    )

Commit message: various fixes
Parts:
- removed J101, J102, J103: Conn_01x03, symbol Connector_Generic:Conn_01x03
- added J101, J102, J103: 705530002, CONN_705530002_03_MOL, symbol misguided:705530002
- added J104: 2601-1102, CONN2_2601-1102_WAG, symbol misguided:2601-1102
Connections:
- net +3.3V: now reaches M101.1 (3v3)
- net +3.3V: now also M101.17 (3v3)
- net OUTPUT: now reaches M101.11 (GPIO17)
- net GND: now reaches M101.14 (GND)
- net GND: now also M101.20 (GND), M101.25 (GND), M101.30 (GND), M101.34 (GND), M101.39 (GND), M101.6 (GND), M101.9 (GND), J104.1 (1_1), J104.2 (1_2)
- net MOSI: now reaches M101.19 (GPIO10)
- net +5V: now reaches M101.2 (5v)
- net +5V: now also M101.4 (5v)
- net MISO: now reaches M101.21 (GPIO09)
- net INT: now reaches M101.22 (GPIO25)
- net CLK: now reaches M101.23 (GPIO11)
- net ~{CS}0: now reaches M101.24 (GPIO08)
- net INPUT: now reaches M101.7 (GPIO04)
- new net +12V: J104.3 (2_1), J104.4 (2_2)
- new net can_bus/CAN_H: J101.3
- new net can_bus/CAN_L: J101.1
- new net dio/DIN: J102.3
- new net dio/DIN_GND: J102.1
- new net dio/DOUT: J103.3
- new net dio/DOUT_GND: J103.1
- new net dio/DOUT_REF: J103.2
- no-connect marks 0 -> 3
Other:
- sheet can_bus ports: added CAN_H, CAN_L, CLK, INT, MISO, MOSI, ~{CS}; removed none
- sheet dio ports: added DIN, DIN_GND, DOUT, DOUT_GND, DOUT_REF, INPUT_GPIO, OUTPUT_GPIO; removed none
- moved on the sheet: M101
