File: misguided/misguided.kicad_sch (KiCad schematic)
At the start: 5 parts, among them J101 705530002, J102 705530002, J103 705530002, J104 2601-1102

Commit message: fixed schematic associations
Parts:
- J101, J102, J103: footprint CONN_705530002_03_MOL -> misguided:CONN_705530002_03_MOL
- J104: footprint CONN2_2601-1102_WAG -> misguided:CONN2_2601-1102_WAG
Changed lines of the file:
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@@
       (effects (font (size 1.524 1.524)) (justify left))
     )
-    (property "Footprint" "CONN2_2601-1102_WAG" (at 41.91 62.23 0)
+    (property "Footprint" "misguided:CONN2_2601-1102_WAG" (at 41.91 62.23 0)
       (effects (font (size 1.27 1.27) italic) hide)
     )
@@
       (effects (font (size 1.524 1.524)) (justify left))
     )
-    (property "Footprint" "CONN_705530002_03_MOL" (at 160.655 84.455 0)
+    (property "Footprint" "misguided:CONN_705530002_03_MOL" (at 160.655 84.455 0)
       (effects (font (size 1.27 1.27) italic) hide)
     )
@@
       (effects (font (size 1.524 1.524)) (justify left))
     )
-    (property "Footprint" "CONN_705530002_03_MOL" (at 177.8 102.235 0)
+    (property "Footprint" "misguided:CONN_705530002_03_MOL" (at 177.8 102.235 0)
       (effects (font (size 1.27 1.27) italic) hide)
     )
@@
       (effects (font (size 1.524 1.524)) (justify left))
     )
-    (property "Footprint" "CONN_705530002_03_MOL" (at 177.8 119.38 0)
-      (effects (font (size 1.27 1.27) italic) hide)
-    )
+    (property "Footprint" "misguided:CONN_705530002_03_MOL" (at 177.8 119.38 0)
+      (effects (font (size 1.27 1.27) italic) hide)
+    )

Commit message: layed out and ordered
Parts:
- added J105: Conn_01x01, misguided:lotion_on_head, symbol Connector_Generic:Conn_01x01
- added J106: Conn_01x01, misguided:robobots, symbol Connector_Generic:Conn_01x01
Connections:
- no-connect marks 24 -> 26
Changed lines of the file:
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@@
   (no_connect (at 73.66 136.525))
   (no_connect (at 73.66 118.745))
+  (no_connect (at 198.12 60.325))
   (no_connect (at 73.66 111.125))
   (no_connect (at 40.64 100.965))
@@
   (no_connect (at 40.64 144.145))
   (no_connect (at 40.64 103.505))
+  (no_connect (at 198.12 54.61))
   (wire (pts (xy 73.66 139.065) (xy 74.93 139.065))
     (stroke (width 0) (type default))
@@
         (path "/2c6152e0-1c3c-4f15-8d1e-fd42bd51bc79"
           (reference "J104") (unit 1)
+        )
+      )
+    )
+  )
+  (symbol (lib_id "Connector_Generic:Conn_01x01") (at 203.2 60.325 0) (unit 1)
+    (in_bom no) (on_board yes) (dnp no) (fields_autoplaced)
+    (property "Reference" "J106" (at 205.74 59.69 0)
+      (effects (font (size 1.27 1.27)) (justify left))
+    )
+    (property "Value" "Conn_01x01" (at 205.74 62.23 0)
+      (effects (font (size 1.27 1.27)) (justify left))
+    )
+    (property "Footprint" "misguided:robobots" (at 203.2 60.325 0)
+      (effects (font (size 1.27 1.27)) hide)
+    )
+    (property "Datasheet" "~" (at 203.2 60.325 0)
+      (effects (font (size 1.27 1.27)) hide)
+    )
+    (pin "1")
+    (instances
+      (project "misguided"
+        (path "/2c6152e0-1c3c-4f15-8d1e-fd42bd51bc79"
+          (reference "J106") (unit 1)
         )
       )
@@
         )
       )
+    )
+  )
+  (symbol (lib_id "Connector_Generic:Conn_01x01") (at 203.2 54.61 0) (unit 1)
+    (in_bom yes) (on_board yes) (dnp no) (fields_autoplaced)
+    (property "Reference" "J105" (at 205.74 53.975 0)
+      (effects (font (size 1.27 1.27)) (justify left))
+    )
+    (property "Value" "Conn_01x01" (at 205.74 56.515 0)
+      (effects (font (size 1.27 1.27)) (justify left))
+    )
+    (property "Footprint" "misguided:lotion_on_head" (at 203.2 54.61 0)
+      (effects (font (size 1.27 1.27)) hide)
+    )
+    (property "Datasheet" "~" (at 203.2 54.61 0)
+      (effects (font (size 1.27 1.27)) hide)
+    )
+    (pin "1")
+    (instances
+      (project "misguided"
+        (path "/2c6152e0-1c3c-4f15-8d1e-fd42bd51bc79"
+          (reference "J105") (unit 1)
+        )
+      )
