File: misguided/power_supplies.kicad_sch (KiCad schematic)
At the start: 0 parts

Commit message: buncha stuff
Parts:
- added U201: MP8756GD-Z, QFN-12_MP8756_MNP, symbol misguided:MP8756GD-Z
Changed lines of the file:
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@@
 (kicad_sch (version 20230121) (generator eeschema)
   (paper "A4")
+  (symbol (lib_id "misguided:MP8756GD-Z") (at 126.365 80.01 0) (unit 1)
+    (in_bom yes) (on_board yes) (dnp no) (fields_autoplaced)
+    (property "Reference" "U201" (at 126.365 76.2 0)
+      (effects (font (size 1.524 1.524)))
+    )
+    (property "Value" "MP8756GD-Z" (at 126.365 78.74 0)
+      (effects (font (size 1.524 1.524)))
+    )
+    (property "Footprint" "QFN-12_MP8756_MNP" (at 126.365 106.045 0)
+      (effects (font (size 1.27 1.27) italic) hide)
+    )
+    (property "Datasheet" "https://www.monolithicpower.com/en/documentview/productdocument/index/version/2/document_type/Datasheet/lang/en/sku/MP8756GD-Z" (at 126.365 102.235 0)
+      (effects (font (size 1.27 1.27) italic) hide)
+    )
+    (pin "1")
+    (pin "10")
+    (pin "11")
+    (pin "12")
+    (pin "2")
+    (pin "3")
+    (pin "4")
+    (pin "5")
+    (pin "6")
+    (pin "7")
+    (pin "8")
+    (pin "9")
+    (instances
+      (project "misguided"
+        (path "/2c6152e0-1c3c-4f15-8d1e-fd42bd51bc79/5c0ad2ae-bc5b-4352-8d7b-34fb763e9c13"
+          (reference "U201") (unit 1)
+        )
+      )
+    )
+  )
 )

Commit message: more setup
Parts:
- renumbered U201 to U?
Changed lines of the file:
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@@
   (symbol (lib_id "misguided:MP8756GD-Z") (at 126.365 80.01 0) (unit 1)
     (in_bom yes) (on_board yes) (dnp no) (fields_autoplaced)
-    (property "Reference" "U201" (at 126.365 76.2 0)
+    (property "Reference" "U?" (at 126.365 76.2 0)
       (effects (font (size 1.524 1.524)))
     )
@@
       (effects (font (size 1.27 1.27) italic) hide)
     )
-    (property "Datasheet" "https://www.monolithicpower.com/en/documentview/productdocument/index/version/2/document_type/Datasheet/lang/en/sku/MP8756GD-Z" (at 126.365 102.235 0)
+    (property "Datasheet" "${KIPRJMOD}/datasheets/MP8756.pdf" (at 126.365 102.235 0)
       (effects (font (size 1.27 1.27) italic) hide)
     )
@@
       (project "misguided"
         (path "/2c6152e0-1c3c-4f15-8d1e-fd42bd51bc79/5c0ad2ae-bc5b-4352-8d7b-34fb763e9c13"
-          (reference "U201") (unit 1)
+          (reference "U?") (unit 1)
         )
       )

Commit message: various fixes
Parts:
- added C201: 22uf, symbol Device:C_Small
- added C202: 1uf, symbol Device:C_Small
- added C203: 220nf, symbol Device:C_Small
- added C204, C205: 100nf, Capacitor_SMD:C_0603_1608Metric, symbol Device:C_Small
- added L201: 3.3uH, Inductor_SMD:L_Coilcraft_XAL7070-XXX, symbol Device:L
- added R201: 3.3, symbol Device:R
- added R202: 110k, symbol Device:R
- added R203: 15k, symbol Device:R
- U?: footprint QFN-12_MP8756_MNP -> misguided:QFN-12_MP8756_MNP
Connections:
- net +12V: now reaches U?.1 (VIN)
- net agnd: now reaches U?.10 (AGND)
- net agnd: now also C202.2
- net at U?.11 (FB): now also R202.2, R203.1
- net GND: now reaches U?.2 (PGND)
- net GND: now also R203.2
- net at U?.7 (SW): now also C203.2, L201.1
- net at U?.8 (BST): now also R201.1
- net at U?.9 (VCC): now also C202.1
- new net: C203.1, R201.2
- new net: L201.2, R202.1
- no-connect marks 0 -> 3

Commit message: schematic finished
Parts:
- added C206, C207, C208, C209, C210, C211, C212: 22uf, Capacitor_SMD:C_0805_2012Metric, symbol Device:C_Small
- added NT201: NetTie_2, symbol Device:NetTie_2
- added R204: 1M, Resistor_SMD:R_0402_1005Metric, symbol Device:R
- added R205: NP, symbol Device:R
- C201: footprint (none) -> Capacitor_SMD:C_0805_2012Metric
Connections:
- net +12V: now also C201.1, C205.1, C206.1, C207.1, C208.1, R204.1
- net GND: now also C201.2, C204.2, C205.2, C206.2, C207.2, C208.2, C209.2, C210.2, C211.2, C212.2, NT201.2
- net agnd: now also NT201.1, R205.2
- net +5V: now reaches C204.1
- net +5V: now also L201.2, R202.1, U?.5 (VOUT), C209.1, C210.1, C211.1, C212.1
- net at U?.12 (EN): now also R204.2, R205.1

Commit message: fixed schematic associations
Parts:
- C211: renamed from C202; footprint (none) -> Capacitor_SMD:C_0603_1608Metric
- C212: renamed from C203; footprint (none) -> Capacitor_SMD:C_0402_1005Metric
- NT201: footprint (none) -> NetTie:NetTie-2_SMD_Pad0.5mm
- R202: renamed from R205; footprint (none) -> Resistor_SMD:R_0402_1005Metric
- R203: renamed from R202; footprint (none) -> Resistor_SMD:R_0402_1005Metric
- R204: renamed from R203; footprint (none) -> Resistor_SMD:R_0402_1005Metric
- R205: renamed from R201; footprint (none) -> Resistor_SMD:R_0402_1005Metric
- gave numbers to parts that had none: 1
- renumbered C204 to C201, C209 to C202, C210 to C203, C211 to C204, C212 to C205, C208 to C206, C201 to C207, C206 to C208, C207 to C209, C205 to C210, R204 to R201

Commit message: layed out and ordered
Parts:
- L201: footprint Inductor_SMD:L_Coilcraft_XAL7070-XXX -> misguided:IND_CYA0630_SHH; PartNumber (none) -> CYA0630-3.3UH
Changed lines of the file:
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@@
       (effects (font (size 1.27 1.27)))
     )
-    (property "Footprint" "Inductor_SMD:L_Coilcraft_XAL7070-XXX" (at 151.765 108.585 0)
+    (property "Footprint" "misguided:IND_CYA0630_SHH" (at 151.765 108.585 0)
       (effects (font (size 1.27 1.27)) hide)
     )
@@
       (effects (font (size 1.27 1.27)) hide)
     )
+    (property "PartNumber" "CYA0630-3.3UH" (at 151.765 108.585 90)
+      (effects (font (size 1.27 1.27)) hide)
+    )
